Commit message: update urdf for depth camera

File: pod2_description/xacro/OpenPodCar_V2_Depth.urdf (robot description, URDF)
Before this commit: robot podcar, 8 links, 7 joints
Links:
- removed link velodyne_link
- added link camera_link, mass 0.01; visual box size=0.01 0.02 0.02

Commit message: Changes to the launch files. Configuartion explaination for navigation. Deleted outdated files.

File: pod2_description/xacro/OpenPodCar_V2_Depth.urdf (robot description, URDF)
Before this commit: robot podcar, 8 links, 7 joints
Joints:
- removed joint velodyne_joint
- added joint camera_joint: type fixed, parent base_link, child camera_link, origin xyz=-0.34 0 1.75 rpy=0 0 0

Commit message: update the packages.

File: pod2_description/xacro/OpenPodCar_V2_Depth.urdf (robot description, URDF)
Before this commit: robot podcar, 8 links, 7 joints
Links:
- added link optical_flow_link, mass 0.01; visual box size=0.01 0.02 0.02
Joints:
- added joint optical_flow_joint: type fixed, parent base_link, child optical_flow_link, origin xyz=+0.0 +0.4 0.155 rpy=0 0 0
- joint camera_joint: origin xyz=-0.34 0 1.75 rpy=0 0 0 -> xyz=+0.8 0 0.68 rpy=0 0 -0.7854
